Commit message: feat(l515): publish color-aligned depth to ROS for RGB-D SLAM (opt-in)
Gateway already produced rs.align color-aligned depth but only fed it to
the SRT streamer, so RTAB-Map had nothing to subscribe to. /l515/depth/* is
raw 640x480 depth in l515_depth_optical_frame while color is 1280x720 in
l515_color_optical_frame, and the two sensors are physically offset, so
their pixels do not correspond — RGB-D SLAM needs depth aligned to color.

Publish it on /l515/aligned_depth_to_color/{image_raw,camera_info} with
frame_id l515_color_optical_frame, taken from the rs frame before it is
flattened to ndarray so the color intrinsics and device timestamp survive.

Off by default: alignment costs CPU (1280x720 warp) and the topics are
heavy. Set L515_ALIGNED_DEPTH_ROS=1 when running SLAM. The existing
six-topic contract and its counts are unchanged when disabled.

_alignment_required() now also returns True when the env flag is set, so
alignment runs for SLAM independently of whether SRT happens to be
streaming in DEPTH/OVERLAY mode.

URDF: L515 mount pitched 15 deg down. Vertical FOV is 55 deg (70 is
horizontal), so 15 deg gives +12.5 / -42.5 coverage — the top stays above
horizontal so walls and pillars remain visible as SLAM features. Pitching
further (25-30) puts the top below horizontal, leaving only floor and
starving SLAM of features. The 0.38 m front blind spot is US-100 territory.
Also adds l515_color_optical_frame, without which rgbd_odometry/rtabmap
fail with "source_frame does not exist".

WIP: depth-color baseline is not yet measured, so the color optical frame
provisionally shares the depth origin (a few mm on L515 — does not affect
pipeline validation, precise calibration to follow).

Co-Authored-By: Claude Opus 4.8 (1M context) <noreply@anthropic.com>

File: ros2/src/powertrain_ros/urdf/jetin_rover.urdf.xacro (robot description, xacro)
@@ -41,4 +41,6 @@
   <xacro:property name="l515_x"  value="0.30"/>
   <xacro:property name="l515_z"  value="0.35"/>
+  <!-- 아래로 숙인 각(+ = 아래). REP-103 에서 pitch + 는 코가 내려가는 방향이다. -->
+  <xacro:property name="l515_pitch_deg" value="15.0"/>
   <xacro:property name="d435i_x" value="0.34"/>
   <xacro:property name="d435i_z" value="0.30"/>
@@ -104,7 +106,14 @@
     </visual>
   </link>
+  <!-- ★ 마운트: 차체 전방, **아래로 15° 숙임** (2026-07-14 설계 확정).
+       왜 15° 인가 — L515 수직화각은 **55°** 다(70° 는 수평). 15° 숙이면 커버리지가
+       상단 +12.5° / 하단 −42.5° 가 된다:
+         · 상단이 **수평 위에 남는다** → 벽·기둥 같은 먼 특징점이 잡힌다. SLAM 이 산다.
+         · 더 숙이면(25~30°) 상단이 수평 아래로 내려가 **바닥만 보게 되고** 특징점이
+           사라져 SLAM 이 망가진다. 사각지대를 줄이려고 숙이면 손해다.
+       앞쪽 0.38 m 는 사각지대 — 어차피 **US-100 이 담당하는 영역**이다. -->
   <joint name="l515_mount" type="fixed">
     <parent link="base_link"/><child link="l515_link"/>
-    <origin xyz="${l515_x} 0 ${l515_z}"/>
+    <origin xyz="${l515_x} 0 ${l515_z}" rpy="0 ${l515_pitch_deg*pi/180} 0"/>
   </joint>
   <!-- depth 토픽의 frame_id. 광학 규약(x=오른쪽, y=아래, z=앞) — 표준 카메라 회전 -->
@@ -112,4 +121,14 @@
   <joint name="l515_optical" type="fixed">
     <parent link="l515_link"/><child link="l515_depth_optical_frame"/>
+    <origin rpy="${-pi/2} 0 ${-pi/2}"/>
+  </joint>
+  <!-- ★ color 광학 프레임 — 정렬(aligned) depth 의 frame_id 가 이거다(gateway_ros.py
+       _COLOR_FRAME). depth-color 베이스라인 실측 전이라 잠정 depth 와 동일 원점으로 둔다
+       (L515 물리 베이스라인은 수 mm 라 SLAM 파이프라인 검증에는 영향 없음 — 정밀 캘리는
+       실측 후 갱신). 이게 없으면 rgbd_odometry/rtabmap 이 "source_frame does not exist" 로
+       계속 실패한다. -->
+  <link name="l515_color_optical_frame"/>
+  <joint name="l515_color_optical" type="fixed">
+    <parent link="l515_link"/><child link="l515_color_optical_frame"/>
     <origin rpy="${-pi/2} 0 ${-pi/2}"/>
   </joint>

Commit message: fix(geometry): take the hardware constants from the as-built v2 CAD
실차 모델(`urdf/urdf_and_usd_v2.zip`, 2026_07_24_URDF + STL 163개)을 직접 재서
코드에 남아 있던 공칭값·v1값·눈대중값을 as-built 실측으로 교체한다. 측정은 URDF
joint chain 의 rpy 를 합성해 STL 정점을 base_link 로 옮기는 방식이고, 원시 STL
바운딩박스로 교차검증했다. base_link 는 로버 중심선에서 x=+0.1200 m 편심,
축거중점 y=+0.353830 m, 지면 z=-0.327240 m 다.

1. 바퀴 반경 0.10 → 0.10356 m
   0.10 은 BL70200 공칭 스펙이었고 실제 타이어 STL 외경은 207.13 mm 다. 이 값은
   원주로 모든 속도 지령과 오도메트리에 곱해지므로 3.4 % 계통오차였다. 무하중
   기하값이며 하중 눌림 실효 반경은 지상 캘리브레이션 몫으로 남는다.
   되돌려도 깨지는 테스트가 하나도 없었으므로 값을 고정하는 테스트를 추가했다.

2. 차폭 팽창 반폭을 타이어에서 허브로 분리 (0.035 → 0.048 m)
   `wheel_half_width_m` 하나가 물리적으로 다른 두 양에 쓰이고 있었다. 접지 밴드는
   타이어 트레드 반폭(±35.0 mm)이 맞지만, 차폭·간극 판정의 외곽 반폭은 인휠 허브가
   결정한다 — 허브 STL 은 같은 축 원점에서 -48.0~+87.0 mm 라 타이어보다 편측
   13 mm 바깥으로 나온다. 로버 전체 메시 bbox 횡폭 0.8150 m 가
   2 × (0.35950 + 0.048) 과 정확히 일치해 교차검증된다.
   → `footprint_outboard_half_width_m` 를 새로 두고 footprint 만 이 값을 쓴다.
   실폭은 0.789 가 아니라 0.815 m 이므로 편측 여유를 13 mm 낙관해온 것이다.

3. `jetin_rover.urdf.xacro` 윤거가 v1 에 머물러 있었다
   0.3525/0.4395/0.2925 → 0.2725/0.3595/0.2125 (윤거 545/719/425 mm). v2 에서
   3030 프로파일이 340→180 mm 로 바뀌며 바퀴가 편측 80 mm 안으로 들어왔는데
   반영이 안 돼 있었다. 파일 주석 스스로 `default_geometry()` 와 같아야 한다고
   적어놓고 어긋나 있었다. 차체 박스 눈대중값(0.80×0.40×0.20 @ z0.30)도 실측
   0.570×0.250×0.250 @ (-0.1038, 0, 0.4472) 로 교체했다.

센서 마운트는 값을 바꾸지 않았다 — v2 URDF/USD 에 카메라·US-100 프림이 아예 없어
도출이 불가능하다. 주석에 그 사실만 기록하고 실측 게이트로 남긴다.

검증: 호스트 943 passed (motor_control + powertrain_autonomy), 변경 전 939 대비
신규 4건(검증 3 + 반경 고정 1)만 증가. 음성 대조 3건 — footprint 배선을 옛 필드로
되돌리면 7건 실패, 상수를 0.035 로 되돌리면 값 고정 테스트 1건 실패, 반경을 0.10 으로
되돌리면 신규 테스트 1건 실패. ROS 컨테이너 colcon 빌드 통과 + xacro 렌더 결과가
`default_geometry()` 와 일치(앞 ±0.2725 / 중 ±0.3595 / 뒤 ±0.2125, wheel_r 0.10356).

⚠️ 이월: `powertrain_sim/assets/rover_model.json` 은 v1 USD 기준이라 stale 하다
   (바퀴 편측 80 mm, 질량 66.96 vs 실제 64.19 kg, 로커한계 ±45° vs 실제 ±20°).
   사용자 지시로 이번엔 sim 을 건드리지 않았다.

Co-Authored-By: Claude Opus 5 (1M context) <noreply@anthropic.com>

File: ros2/src/powertrain_ros/urdf/jetin_rover.urdf.xacro (robot description, xacro)
@@ -4,17 +4,16 @@
     확인:  xacro jetin_rover.urdf.xacro > /tmp/out.urdf && check_urdf /tmp/out.urdf
     사용:  ros2 launch powertrain_ros robot_viz.launch.py
-  ⚠️ **이것은 시각화·TF 용 최소 모델이다.** 실물 CAD 형상이 아니다.
+  ⚠️ **이것은 시각화·TF 용 최소 모델이다.** 실물 CAD 메시 모델이 아니다.
      로커·보기 링키지, 서스펜션, 로봇팔은 없다. 목적은 오직 두 가지 —
        ① RViz 에서 로봇의 자세·바퀴·조향을 눈으로 본다
        ② `base_link → 각 바퀴/센서` TF 를 robot_state_publisher 가 자동 생성한다
-     설계팀 정본 URDF 가 오면 이 파일을 갈아끼운다. 그때까지 파이프라인을 막지 않는다.
+     바퀴·차체 치수는 as-built v2 CAD 실측을 반영했다. 센서 마운트만 v2 CAD 에도
+     형상이 없어 실측 게이트로 남아 있다(2026-08-01 확인).
   ── 치수 출처 ──────────────────────────────────────────────────────────────
-  · 바퀴 x (앞뒤)  = **v4 최적화 설계값**. `parameter_calc/python_gpu_triangle/
-    export_chassis_geometry.py` 가 정본 pkl(f_opt 0.2004)에서 평지 접지 평형을 풀어 도출.
+  · 바퀴 중심·타이어·차체 박스 = **as-built v2 CAD 실측**.
     `motor_control/chassis/kinematics.py` 의 `default_geometry()` 와 **같은 숫자여야 한다.**
-  · 바퀴 반경 0.10 m = R_w (v4 · BL70200 인휠).
-  · 윤거(좌우) = ⚠️ **근거 없음 — 설계팀 실측 대기.** v4 는 측면-절반 2D 모델이라
-    좌우 치수를 아예 다루지 않는다. 실측이 오면 `track_half` 만 바꾸면 된다.
-  · 차체 박스·센서 마운트 = ⚠️ **눈대중 플레이스홀더.**
+  · 바퀴 반경 0.10356 m = 타이어 STL 외경 207.13 mm 의 무하중 기하값.
+  · 윤거(좌우) = 앞 545 / 중간 719 / 뒤 425 mm. 허브 외측 돌출을 포함한 차폭은 815 mm.
+  · 차체 박스는 as-built 실측이며, 센서 마운트만 ⚠️ **미실측 플레이스홀더.**
 -->
 <robot name="jetin_rover" xmlns:xacro="http://www.ros.org/wiki/xacro">
@@ -22,5 +21,5 @@
   <!-- **설계팀 CAD URDF 실측** — scripts/extract_geometry_from_cad_urdf.py
        kinematics.default_geometry() 와 **같은 숫자여야 한다.**
-       ⚠️ 윤거가 앞/중/뒤 전부 다르다 (705 / 879 / 585 mm). CAD 상 실측이며 오독이 아니다
+       ⚠️ 윤거가 앞/중/뒤 전부 다르다 (545 / 719 / 425 mm). CAD 상 실측이며 오독이 아니다
           (조향 4륜의 타이어 원점이 킹핀 축과 Δ0.0 mm 일치 = 스크럽 반경 0 설계).
           **설계 의도인지 CAD 오류인지 설계팀 확인 필요.** -->
@@ -28,15 +27,18 @@
   <xacro:property name="x_mid"      value="-0.0603"/>  <!-- ⚠️ 축거중심에서 60 mm 뒤 -->
   <xacro:property name="x_rear"     value="-0.4377"/>
-  <xacro:property name="y_front"    value="0.3525"/>   <!-- 앞 윤거 705 mm -->
-  <xacro:property name="y_mid"      value="0.4395"/>   <!-- 중간 윤거 879 mm -->
-  <xacro:property name="y_rear"     value="0.2925"/>   <!-- 뒤 윤거 585 mm -->
-  <xacro:property name="wheel_r"    value="0.10"/>
+  <xacro:property name="y_front"    value="0.2725"/>   <!-- 앞 윤거 545 mm -->
+  <xacro:property name="y_mid"      value="0.3595"/>   <!-- 중간 윤거 719 mm -->
+  <xacro:property name="y_rear"     value="0.2125"/>   <!-- 뒤 윤거 425 mm -->
+  <xacro:property name="wheel_r"    value="0.10356"/>
   <xacro:property name="wheel_w"    value="0.07"/>   <!-- 타이어 폭 70 mm -->
-  <!-- ⚠️ 차체 박스는 눈대중 플레이스홀더 (CAD 메시가 오면 교체) -->
-  <xacro:property name="body_l"     value="0.80"/>
-  <xacro:property name="body_w"     value="0.40"/>
-  <xacro:property name="body_h"     value="0.20"/>
-  <xacro:property name="body_z"     value="0.30"/>   <!-- 지면 위 차체 높이 -->
-  <!-- ⚠️ 센서 마운트 = 미실측. imu_tilt_node 의 mount_* 기본값과 맞춰둠 -->
+  <!-- as-built v2 CAD 실측 차체 프레임 박스. 3030+판재 기준 폭 250 mm,
+       로커피벗 보스 포함 폭 470 mm, 전체 외곽 포락 1083 × 815 × 604 mm. -->
+  <xacro:property name="body_l"     value="0.570"/>
+  <xacro:property name="body_w"     value="0.250"/>
+  <xacro:property name="body_h"     value="0.250"/>
+  <xacro:property name="body_x"     value="-0.1038"/> <!-- 축거중점 기준 박스 중심 -->
+  <xacro:property name="body_z"     value="0.4472"/>  <!-- 지면 위 박스 중심 -->
+  <!-- ⚠️ 센서 마운트 = v2 CAD 에 센서 형상 없음 — 실측 게이트(2026-08-01 확인).
+       imu_tilt_node 의 mount_* 기본값과 맞춰둠. -->
   <xacro:property name="l515_x"  value="0.30"/>
   <xacro:property name="l515_z"  value="0.35"/>
@@ -52,5 +54,5 @@
   <link name="base_link">
     <visual>
-      <origin xyz="0 0 ${body_z}"/>
+      <origin xyz="${body_x} 0 ${body_z}"/>
       <geometry><box size="${body_l} ${body_w} ${body_h}"/></geometry>
       <material name="grey"/>
